Commit message: fix: 修正wc4把手坐标轴错误，优化门json配置

File: high-level/data/asset/door_set/wc4/model.urdf (robot description, URDF)
Before this commit: robot single_leaf_restroom_door, 8 links, 7 joints
Links:
- link lever_handle: geometry collision box size=0.02 0.03 0.01; collision box size=0.12 0.02 0.01
Joints:
- joint handle_spindle_joint: axis 0 -1 0 -> 0 0 1; origin xyz=0 -0.013 0 rpy=0 0 0 -> xyz=0 -0.013 0 rpy=1.5707963267948966 0 0

Commit message: 深度图修改 调整分辨率 增加噪声

File: high-level/data/asset/door_set/wc4/model.urdf (robot description, URDF)
Before this commit: robot single_leaf_restroom_door, 8 links, 7 joints
Links:
- link lever_handle: geometry collision box size=0.02 0.03 0.01; collision box size=0.12 0.02 0.01
