Commit message: Float IK: left-push 成功

File: high-level/data/asset/door_set/record_materialization/rec_using-the-reference-image-for-overall-proportion_20260610_185617_636160_746172d9/model.urdf (robot description, URDF)
Before this commit: robot burgundy_single_leaf_door, 6 links, 5 joints
Joints:
- joint handle_actuation_joint: limit lower=0 upper=0.523599 effort=3 velocity=2 -> lower=0 upper=1.5707963267948966 effort=3 velocity=2
