Commit message: fix: 修正a2wz1为整体资产直接加载，不进行分体flip操作

File: high-level/data/asset/a2wz1/urdf/a2wz1.urdf (robot description, URDF)
Before this commit: robot a2wz1, 31 links, 30 joints
Links:
- link gripperMover: geometry collision mesh filename=../meshes/z1_GripperMover.dae scale=1 1 1; visual mesh filename=../meshes/z1_GripperMover.dae scale=1 1 1
- link gripperStator: geometry collision mesh filename=../meshes/z1_GripperStator.dae scale=1 1 1; visual mesh filename=../meshes/z1_GripperStator.dae scale=1 1 1
- link link00: geometry collision cylinder length=0.03 radius=0.0325; visual mesh filename=../meshes/z1_Link00.dae scale=1 1 1
- link link02: geometry collision cylinder length=0.051 radius=0.0325; collision cylinder length=0.102 radius=0.02
- link link04: geometry collision cylinder length=0.073 radius=0.0325; visual mesh filename=../meshes/z1_Link04.dae scale=1 1 1
Joints:
- joint base_static_joint: origin xyz=0.20 0 0.1 rpy=0 0 0 -> xyz=0.3 0 0.09 rpy=0 0 0
- joint joint1: limit lower=-2.618 upper=2.618 effort=30.0 velocity=10 -> lower=-2.6179938779914944 upper=2.6179938779914944 effort=30.0 velocity=10
- joint joint2: limit lower=0.0 upper=3.14 effort=60.0 velocity=10 -> lower=0.0 upper=3.141592653589793 effort=60.0 velocity=10
- joint joint3: limit lower=-4.78 upper=0.0 effort=30.0 velocity=10 -> lower=-4.782202150464463 upper=0.0 effort=30.0 velocity=10
- joint joint4: limit lower=-1.744 upper=1.57 effort=30.0 velocity=10 -> lower=-1.7453292519943295 upper=1.5707963267948966 effort=30.0 velocity=10
- joint joint5: limit lower=-1.727 upper=1.727 effort=30.0 velocity=10 -> lower=-1.7278759594743864 upper=1.7278759594743864 effort=30.0 velocity=10
- joint joint6: limit lower=-2.79 upper=2.79 effort=30.0 velocity=10 -> lower=-2.792526803190927 upper=2.792526803190927 effort=30.0 velocity=10
- joint jointGripper: limit lower=-1.57 upper=0.0 effort=30.0 velocity=10 -> lower=-1.5707963267948966 upper=0.0 effort=30.0 velocity=10

Commit message: 1 新增 A2W+Z1 开门仿真主流程 2 新增 A2W 数据录制脚本 3 深度图和噪声流程改了 4 Door / robot 随机化和轨迹默认改了 门和墙体逻辑修了 5 eval/play 新增 A2W 入口 6 新增实机部署相关目录

File: high-level/data/asset/a2wz1/urdf/a2wz1.urdf (robot description, URDF)
Before this commit: robot a2wz1, 31 links, 30 joints
Joints:
- joint base_static_joint: origin xyz=0.20 0 0.1 rpy=0 0 0 -> xyz=0.174 0 0.142 rpy=0 0 0
