Commit message: 修改相机配置、相机支架、深度图噪声、支持9D数据
Co-authored-by: Copilot <copilot@github.com>

File: high-level/data/asset/a2wz1/urdf/a2wz1.urdf (robot description, URDF)
Before this commit: robot a2wz1, 31 links, 30 joints
Links:
- added link wrist_down_mount, mass 0.001; collision mesh filename=../meshes/wrist_mount_up.STL scale=1 1 1; visual mesh filename=../meshes/wrist_mount_up.STL scale=1 1 1
- added link wrist_up_mount, mass 0.001; collision mesh filename=../meshes/wrist_mount_down.STL scale=1 1 1; visual mesh filename=../meshes/wrist_mount_down.STL scale=1 1 1
Joints:
- added joint wrist_down_mount_joint: type fixed, parent link06, child wrist_down_mount, origin xyz=0.065 0 0 rpy=-1.5707963267948966 0 0
- added joint wrist_up_mount_joint: type fixed, parent link06, child wrist_up_mount, origin xyz=0.035 0 0 rpy=-1.5707963267948966 0 0
